File: MiniProject1/MiniProject1Good.kicad_pcb (KiCad board)
At the start: 2 copper layers, 25.4 x 25.4 mm, 23 parts, among them J1 USB_A, U1 LinearReg, U2 OpAmp, U3 OpAmp

Commit message: Fixed bypass caps
Connections:
- C1 pad 2: Net-(C1-Pad2) -> GND
- C2 pad 2: Net-(C2-Pad2) -> GND
- J1 pad 1: Net-(C1-Pad2) -> Net-(C1-Pad1)
- R1 pad 1: Net-(C2-Pad2) -> Net-(C2-Pad1)
Routing:
- net GND: track 87.6 -> 96.3 mm
- net Net-(C2-Pad1): track 4.03 -> 10.8 mm
- net Net-(C1-Pad2): track 6.75 -> 0.00 mm
- net Net-(C2-Pad2): track 3.47 -> 0.00 mm
- net Net-(C1-Pad1): track 6.87 -> 8.38 mm
