File: MiniProject1/MiniProject1.sch (KiCad schematic (older format))
At the start: 23 parts, among them J1 USB_A, U1 LinearReg, U2 OpAmp, U3 OpAmp

Commit message: Fixed RC values
Connections:
- net GND: now also C1.2, C2.2
- net at R1.1: now also C2.1, U1.2 (Vout); no longer C2.2
- net at J1.1 (VBUS): now also C1.1, U1.3 (Vin); no longer C1.2
Changed lines of the file:
@@
 	1950 2250 2350 2250
-Wire Wire Line
-	1600 2400 1900 2400
-Wire Wire Line
-	1900 2400 1900 2750
-Wire Wire Line
-	1900 2750 2350 2750
-Wire Wire Line
-	3250 2750 2750 2750
-Wire Wire Line
-	2750 2750 2750 3500
-Wire Wire Line
-	2750 3500 2200 3500
 Wire Wire Line
 	2200 3500 2200 3700
@@
 	1    0    0    -1
 $EndComp
+Wire Wire Line
+	2350 2400 2350 2450
+Wire Wire Line
+	1600 2400 2350 2400
+Connection ~ 2350 2450
+Wire Wire Line
+	3250 2450 3750 2450
+Wire Wire Line
+	3750 2450 3750 2850
+Wire Wire Line
+	3750 2850 2900 2850
+Wire Wire Line
+	2900 2850 2900 3500
+Wire Wire Line
+	2200 3500 2900 3500
+Connection ~ 3250 2450
+$Comp
+L power:GND #PWR0101
+U 1 1 5C61ABD5
+P 2350 2750
+F 0 "#PWR0101" H 2350 2500 50  0001 C CNN
+F 1 "GND" H 2355 2577 50  0000 C CNN
+F 2 "" H 2350 2750 50  0001 C CNN
+F 3 "" H 2350 2750 50  0001 C CNN
+	1    2350 2750
+	1    0    0    -1
+$EndComp
+$Comp
+L power:GND #PWR0102
+U 1 1 5C61AC25
+P 3250 2750
+F 0 "#PWR0102" H 3250 2500 50  0001 C CNN
+F 1 "GND" H 3255 2577 50  0000 C CNN
+F 2 "" H 3250 2750 50  0001 C CNN
+F 3 "" H 3250 2750 50  0001 C CNN
+	1    3250 2750
+	1    0    0    -1
+$EndComp
